File: PCBs/Amplificador Simple de Dos Etapas/Amplificador Simple de Dos Etapas.kicad_sch (KiCad schematic)
At the start: 14 parts, among them Q1 2N331, Q2 2N331

Commit message: Se hizo una revisión al circuito del amplificador simple, se logró hacer que funcione con transistores modernos 2N3906.
Parts:
- B1: value 4.5 -> 9
- Q1, Q2: value 2N331 -> 2N3906
- R1: value 180k -> 220k
- R3: value 180k -> 100k
- R7: value 1k -> 470
Other:
- note added: ".control * 1. Ejecutar la simulacion (10ms da tiempo a que la onda se estabilice) tran 10u 10m * 2. Medir voltajes (ignorar los primeros 2ms del arranque) meas tran v_in_pp PP V(Entrada_-) FROM=2m meas tran v_out_pp PP V(Salida_-) FROM=2m * 3. Calcular ganancia let ganancia_calculada = v_out_pp / v_in_pp * 4. Crear un separador visual para la consola echo "" echo "================================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"
Changed lines of the file:
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@@
+		)
+	)
+	(text ".control\n  * 1. Ejecutar la simulacion (10ms da tiempo a que la onda se estabilice)\n  tran 10u 10m\n  \n  * 2. Medir voltajes (ignorar los primeros 2ms del arranque)\n  meas tran v_in_pp PP V(Entrada_-) FROM=2m\n  meas tran v_out_pp PP V(Salida_-) FROM=2m\n  \n  * 3. Calcular ganancia\n  let ganancia_calculada = v_out_pp / v_in_pp\n  \n  * 4. Crear un separador visual para la consola\n  echo \"\"\n  echo \"==================================================\"\n  echo \"      RESULTADOS DE RENDIMIENTO Y DISTORSION      \"\n  echo \"==================================================\"\n  \n  * 5. Imprimir la ganancia\n  print ganancia_calculada\n  \n  * 6. Calcular Distorsion Armonica Total (THD) a 1kHz\n  echo \"--------------------------------------------------\"\n  fourier 1k V(Salida_-)\n  \n  echo \"==================================================\"\n.endc"
+		(exclude_from_sim no)
+		(at 54.864 121.158 0)
+		(effects
+			(font
+				(size 1.27 1.27)
+			)
 		)
 	)
@@
 	)
 	(junction
-		(at 99.06 29.21)
+		(at 101.6 54.61)
 		(diameter 0)
 		(color 0 0 0 0)
 	)
 	(junction
-		(at 95.25 54.61)
+		(at 99.06 29.21)
 		(diameter 0)
 		(color 0 0 0 0)
@@
 	(wire
 		(pts
+			(xy 101.6 54.61) (xy 99.06 54.61)
+		)
+		(stroke
+			(width 0)
+			(type default)
+		)
+	)
+	(wire
+		(pts
 			(xy 50.8 29.21) (xy 62.23 29.21)
 		)
@@
 	(wire
 		(pts
-			(xy 95.25 54.61) (xy 99.06 54.61)
-		)
-		(stroke
-			(width 0)
-			(type default)
-		)
-	)
-	(wire
-		(pts
-			(xy 62.23 54.61) (xy 95.25 54.61)
+			(xy 62.23 54.61) (xy 99.06 54.61)
 		)
 		(stroke
@@
 	(wire
 		(pts
+			(xy 101.6 54.61) (xy 102.87 54.61)
+		)
+		(stroke
+			(width 0)
+			(type default)
+		)
+	)
+	(wire
+		(pts
 			(xy 62.23 39.37) (xy 62.23 40.64)
 		)
@@
 	(wire
 		(pts
-			(xy 99.06 54.61) (xy 102.87 54.61)
-		)
-		(stroke
-			(width 0)
-			(type default)
-		)
-	)
-	(wire
-		(pts
 			(xy 49.53 46.99) (xy 50.8 46.99)
 		)
@@
 	(wire
 		(pts
-			(xy 95.25 54.61) (xy 95.25 55.88)
+			(xy 101.6 54.61) (xy 101.6 55.88)
 		)
 		(stroke
@@
 			)
 		)
-		(property "Value" "2N331"
+		(property "Value" "2N3906"
 			(at 101.6 48.2599 0)
 			(effects
@@
 			)
 		)
+		(property "Sim.Library" "/home/martiagosantinez/Desktop/Github/ABC_del_Joven_Radiotecnico/ABC-del-Joven-Radiotecnico/PCBs/2N3906.lib"
+			(at 96.52 46.99 0)
+			(effects
+				(font
+					(size 1.27 1.27)
+				)
+				(hide yes)
+			)
+		)
+		(property "Sim.Name" "2N3906"
+			(at 96.52 46.99 0)
+			(effects
+				(font
+					(size 1.27 1.27)
+				)
+				(hide yes)
+			)
+		)
 		(property "Sim.Device" "PNP"
-			(at 96.52 46.99 0)
-			(effects
-				(font
-					(size 1.27 1.27)
-				)
-				(hide yes)
-			)
-		)
-		(property "Sim.Library" "2n331.lib"
-			(at 96.52 46.99 0)
-			(effects
-				(font
-					(size 1.27 1.27)
-				)
-				(hide yes)
-			)
-		)
-		(property "Sim.Name" "2N331"
 			(at 96.52 46.99 0)
 			(effects
@@
 			)
 		)
-		(property "Value" "2N331"
+		(property "Value" "2N3906"
 			(at 64.77 48.2599 0)
 			(effects
@@
 			)
 		)
-		(property "Sim.Library" "2n331.lib"
+		(property "Sim.Library" "/home/martiagosantinez/Desktop/Github/ABC_del_Joven_Radiotecnico/ABC-del-Joven-Radiotecnico/PCBs/2N3906.lib"
 			(at 59.69 46.99 0)
 			(effects
@@
 			)
 		)
-		(property "Sim.Name" "2N331"
+		(property "Sim.Name" "2N3906"
 			(at 59.69 46.99 0)
 			(effects
@@
 			)
 		)
-		(property "Value" "180k"
+		(property "Value" "220k"
 			(at 53.34 34.2899 0)
 			(effects
@@
 			)
 		)
-		(property "Value" "4.5"
+		(property "Value" "9"
 			(at 49.53 73.6599 0)
 			(effects
@@
 			)
 		)
-		(property "Value" "180k"
+		(property "Value" "100k"
 			(at 91.44 34.2899 0)
 			(effects
@@
 	(symbol
 		(lib_id "Simulation_SPICE:0")
-		(at 95.25 55.88 0)
+		(at 101.6 55.88 0)
 		(unit 1)
 		(exclude_from_sim no)
@@
 		(fields_autoplaced yes)
 		(property "Reference" "#GND01"
-			(at 95.25 60.96 0)
+			(at 101.6 60.96 0)
 			(effects
 				(font
@@
 		)
 		(property "Value" "0"
-			(at 95.25 53.34 0)
+			(at 101.6 53.34 0)
 			(effects
 				(font
@@
 		)
 		(property "Footprint" ""
-			(at 95.25 55.88 0)
+			(at 101.6 55.88 0)
 			(effects
 				(font
@@
 		)
 		(property "Datasheet" "https://ngspice.sourceforge.io/docs/ngspice-html-manual/manual.xhtml#subsec_Circuit_elements__device"
-			(at 95.25 66.04 0)
+			(at 101.6 66.04 0)
 			(effects
 				(font
@@
 		)
 		(property "Description" "0V reference potential for simulation"
-			(at 95.25 63.5 0)
+			(at 101.6 63.5 0)
 			(effects
 				(font
@@
 			)
 		)
-		(property "Value" "1k"
+		(property "Value" "470"
 			(at 71.1199 38.1 0)
 			(effects
